File: Projet commun SEC SIC/Projet commun SEC SIC-PAS TOUT.kicad_pcb (KiCad board)
At the start: 2 copper layers, 249.5 x 112.5 mm, 4 parts, among them J1 Conn_01x08_Female, J2 Conn_01x06_Female, J3 Conn_01x09_Female, U1 ATmega328-P

Commit message: placement elements PCB
Parts:
- moved J2 172.7 mm to (88.0, 68.0)
- moved J1 164.9 mm to (92.1, 97.6), turned to 180 degrees
- moved U1 58.5 mm to (56.5, 69.0)
- moved J3 35.0 mm to (37.2, 74.4), turned to 180 degrees
Routing:
- net Net-(J1-Pad2): track 0.00 -> 29.7 mm
- net Net-(J1-Pad5): track 0.00 -> 28.7 mm
- net Net-(J1-Pad3): track 0.00 -> 28.5 mm
- net Net-(J1-Pad4): track 0.00 -> 28.0 mm
- net Net-(J2-Pad3): track 0.00 -> 24.5 mm
- net Net-(J2-Pad2): track 0.00 -> 23.9 mm
- net Net-(J3-Pad5): track 0.00 -> 20.8 mm
- net Net-(J3-Pad6): track 0.00 -> 20.2 mm
Changed lines of the file:
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@@
   (net 36 "unconnected-(J2-Pad5)")
   (footprint "Package_DIP:DIP-28_W7.62mm" placed (layer "F.Cu")
-    (at 113.7 81.5)
+    (at 56.525 68.971)
     (descr "28-lead though-hole mounted DIP package, row spacing 7.62 mm (300 mils)")
     (tags "THT DIP DIL PDIP 2.54mm 7.62mm 300mil")
@@
   )
   (footprint "Connector_PinHeader_1.00mm:PinHeader_1x09_P1.00mm_Vertical" placed (layer "F.Cu")
-    (at 40 39.5)
+    (at 37.211 74.358 180)
     (descr "Through hole straight pin header, 1x09, 1.00mm pitch, single row")
     (tags "Through hole pin header THT 1x09 1.00mm single row")
@@
     (fp_line (start -0.635 -0.1825) (end -0.3175 -0.5) (layer "F.Fab") (width 0.1))
     (fp_line (start 0.635 -0.5) (end 0.635 8.5) (layer "F.Fab") (width 0.1))
-    (pad "1" thru_hole rect (at 0 0) (size 0.85 0.85) (drill 0.5) (layers *.Cu *.Mask)
+    (pad "1" thru_hole rect (at 0 0 180) (size 0.85 0.85) (drill 0.5) (layers *.Cu *.Mask)
       (net 28 "unconnected-(J3-Pad1)") (pinfunction "Pin_1") (pintype "passive+no_connect"))
-    (pad "2" thru_hole oval (at 0 1) (size 0.85 0.85) (drill 0.5) (layers *.Cu *.Mask)
+    (pad "2" thru_hole oval (at 0 1 180) (size 0.85 0.85) (drill 0.5) (layers *.Cu *.Mask)
       (net 29 "unconnected-(J3-Pad2)") (pinfunction "Pin_2") (pintype "passive+no_connect"))
-    (pad "3" thru_hole oval (at 0 2) (size 0.85 0.85) (drill 0.5) (layers *.Cu *.Mask)
+    (pad "3" thru_hole oval (at 0 2 180) (size 0.85 0.85) (drill 0.5) (layers *.Cu *.Mask)
       (net 30 "unconnected-(J3-Pad3)") (pinfunction "Pin_3") (pintype "passive+no_connect"))
-    (pad "4" thru_hole oval (at 0 3) (size 0.85 0.85) (drill 0.5) (layers *.Cu *.Mask)
+    (pad "4" thru_hole oval (at 0 3 180) (size 0.85 0.85) (drill 0.5) (layers *.Cu *.Mask)
       (net 31 "unconnected-(J3-Pad4)") (pinfunction "Pin_4") (pintype "passive+no_connect"))
-    (pad "5" thru_hole oval (at 0 4) (size 0.85 0.85) (drill 0.5) (layers *.Cu *.Mask)
+    (pad "5" thru_hole oval (at 0 4 180) (size 0.85 0.85) (drill 0.5) (layers *.Cu *.Mask)
       (net 3 "Net-(J3-Pad5)") (pinfunction "Pin_5") (pintype "passive"))
-    (pad "6" thru_hole oval (at 0 5) (size 0.85 0.85) (drill 0.5) (layers *.Cu *.Mask)
+    (pad "6" thru_hole oval (at 0 5 180) (size 0.85 0.85) (drill 0.5) (layers *.Cu *.Mask)
       (net 2 "Net-(J3-Pad6)") (pinfunction "Pin_6") (pintype "passive"))
-    (pad "7" thru_hole oval (at 0 6) (size 0.85 0.85) (drill 0.5) (layers *.Cu *.Mask)
+    (pad "7" thru_hole oval (at 0 6 180) (size 0.85 0.85) (drill 0.5) (layers *.Cu *.Mask)
       (net 8 "GND") (pinfunction "Pin_7") (pintype "passive"))
-    (pad "8" thru_hole oval (at 0 7) (size 0.85 0.85) (drill 0.5) (layers *.Cu *.Mask)
+    (pad "8" thru_hole oval (at 0 7 180) (size 0.85 0.85) (drill 0.5) (layers *.Cu *.Mask)
       (net 7 "VCC") (pinfunction "Pin_8") (pintype "passive"))
-    (pad "9" thru_hole oval (at 0 8) (size 0.85 0.85) (drill 0.5) (layers *.Cu *.Mask)
+    (pad "9" thru_hole oval (at 0 8 180) (size 0.85 0.85) (drill 0.5) (layers *.Cu *.Mask)
       (net 32 "unconnected-(J3-Pad9)") (pinfunction "Pin_9") (pintype "passive"))
     (model "${KICAD6_3DMODEL_DIR}/Connector_PinHeader_1.00mm.3dshapes/PinHeader_1x09_P1.00mm_Vertical.wrl"
@@
   )
   (footprint "Connector_PinHeader_1.00mm:PinHeader_1x06_P1.00mm_Vertical" placed (layer "F.Cu")
-    (at 256.5 30)
+    (at 88.011 67.985)
     (descr "Through hole straight pin header, 1x06, 1.00mm pitch, single row")
     (tags "Through hole pin header THT 1x06 1.00mm single row")
@@
   )
   (footprint "Connector_PinHeader_1.00mm:PinHeader_1x08_P1.00mm_Vertical" placed (layer "F.Cu")
-    (at 256.5 110.5)
+    (at 92.075 97.592 180)
     (descr "Through hole straight pin header, 1x08, 1.00mm pitch, single row")
     (tags "Through hole pin header THT 1x08 1.00mm single row")
@@
     (fp_line (start -0.635 -0.1825) (end -0.3175 -0.5) (layer "F.Fab") (width 0.1))
     (fp_line (start -0.635 7.5) (end -0.635 -0.1825) (layer "F.Fab") (width 0.1))
-    (pad "1" thru_hole rect (at 0 0) (size 0.85 0.85) (drill 0.5) (layers *.Cu *.Mask)
+    (pad "1" thru_hole rect (at 0 0 180) (size 0.85 0.85) (drill 0.5) (layers *.Cu *.Mask)
       (net 33 "unconnected-(J1-Pad1)") (pinfunction "Pin_1") (pintype "passive+no_connect"))
-    (pad "2" thru_hole oval (at 0 1) (size 0.85 0.85) (drill 0.5) (layers *.Cu *.Mask)
+    (pad "2" thru_hole oval (at 0 1 180) (size 0.85 0.85) (drill 0.5) (layers *.Cu *.Mask)
       (net 16 "Net-(J1-Pad2)") (pinfunction "Pin_2") (pintype "passive"))
-    (pad "3" thru_hole oval (at 0 2) (size 0.85 0.85) (drill 0.5) (layers *.Cu *.Mask)
+    (pad "3" thru_hole oval (at 0 2 180) (size 0.85 0.85) (drill 0.5) (layers *.Cu *.Mask)
       (net 17 "Net-(J1-Pad3)") (pinfunction "Pin_3") (pintype "passive"))
-    (pad "4" thru_hole oval (at 0 3) (size 0.85 0.85) (drill 0.5) (layers *.Cu *.Mask)
+    (pad "4" thru_hole oval (at 0 3 180) (size 0.85 0.85) (drill 0.5) (layers *.Cu *.Mask)
       (net 18 "Net-(J1-Pad4)") (pinfunction "Pin_4") (pintype "passive"))
-    (pad "5" thru_hole oval (at 0 4) (size 0.85 0.85) (drill 0.5) (layers *.Cu *.Mask)
+    (pad "5" thru_hole oval (at 0 4 180) (size 0.85 0.85) (drill 0.5) (layers *.Cu *.Mask)
       (net 19 "Net-(J1-Pad5)") (pinfunction "Pin_5") (pintype "passive"))
-    (pad "6" thru_hole oval (at 0 5) (size 0.85 0.85) (drill 0.5) (layers *.Cu *.Mask)
+    (pad "6" thru_hole oval (at 0 5 180) (size 0.85 0.85) (drill 0.5) (layers *.Cu *.Mask)
       (net 8 "GND") (pinfunction "Pin_6") (pintype "passive"))
-    (pad "7" thru_hole oval (at 0 6) (size 0.85 0.85) (drill 0.5) (layers *.Cu *.Mask)
+    (pad "7" thru_hole oval (at 0 6 180) (size 0.85 0.85) (drill 0.5) (layers *.Cu *.Mask)
       (net 34 "unconnected-(J1-Pad7)") (pinfunction "Pin_7") (pintype "passive+no_connect"))
-    (pad "8" thru_hole oval (at 0 7) (size 0.85 0.85) (drill 0.5) (layers *.Cu *.Mask)
+    (pad "8" thru_hole oval (at 0 7 180) (size 0.85 0.85) (drill 0.5) (layers *.Cu *.Mask)
       (net 7 "VCC") (pinfunction "Pin_8") (pintype "passive"))
     (model "${KICAD6_3DMODEL_DIR}/Connector_PinHeader_1.00mm.3dshapes/PinHeader_1x08_P1.00mm_Vertical.wrl"
@@
   )
   (gr_rect (start 21 19) (end 270.5 131.5) (layer "Edge.Cuts") (width 0.1) (fill none))
+  (segment (start 48.53 69.358) (end 50.683 71.511) (width 0.25) (layer "F.Cu") (net 2))
+  (segment (start 50.683 71.511) (end 56.525 71.511) (width 0.25) (layer "F.Cu") (net 2))
+  (segment (start 37.211 69.358) (end 48.53 69.358) (width 0.25) (layer "F.Cu") (net 2))
+  (segment (start 50.048 74.051) (end 56.525 74.051) (width 0.25) (layer "F.Cu") (net 3))
+  (segment (start 37.211 70.358) (end 46.355 70.358) (width 0.25) (layer "F.Cu") (net 3))
+  (segment (start 46.355 70.358) (end 50.048 74.051) (width 0.25) (layer "F.Cu") (net 3))
+  (segment (start 86.868 97.663) (end 86.868 96.647) (width 0.25) (layer "F.Cu") (net 16))
+  (segment (start 85.08 99.451) (end 86.868 97.663) (width 0.25) (layer "F.Cu") (net 16))
+  (segment (start 86.923 96.592) (end 92.075 96.592) (width 0.25) (layer "F.Cu") (net 16))
+  (segment (start 64.145 99.451) (end 85.08 99.451) (width 0.25) (layer "F.Cu") (net 16))
+  (segment (start 86.868 96.647) (end 86.923 96.592) (width 0.25) (layer "F.Cu") (net 16))
+  (segment (start 79.033 95.592) (end 92.075 95.592) (width 0.25) (layer "F.Cu") (net 17))
+  (segment (start 77.714 96.911) (end 79.033 95.592) (width 0.25) (layer "F.Cu") (net 17))
+  (segment (start 64.145 96.911) (end 77.714 96.911) (width 0.25) (layer "F.Cu") (net 17))
+  (segment (start 64.145 94.371) (end 91.854 94.371) (width 0.25) (layer "F.Cu") (net 18))
+  (segment (start 91.854 94.371) (end 92.075 94.592) (width 0.25) (layer "F.Cu") (net 18))
+  (segment (start 76.845 91.831) (end 78.613 93.599) (width 0.25) (layer "F.Cu") (net 19))
+  (segment (start 78.613 93.599) (end 78.62 93.592) (width 0.25) (layer "F.Cu") (net 19))
+  (segment (start 64.145 91.831) (end 76.845 91.831) (width 0.25) (layer "F.Cu") (net 19))
+  (segment (start 78.62 93.592) (end 92.075 93.592) (width 0.25) (layer "F.Cu") (net 19))
+  (segment (start 64.145 71.511) (end 77.968 71.511) (width 0.25) (layer "F.Cu") (net 26))
+  (segment (start 77.968 71.511) (end 79.502 69.977) (width 0.25) (layer "F.Cu") (net 26))
+  (segment (start 79.51 69.985) (end 88.011 69.985) (width 0.25) (layer "F.Cu") (net 26))
+  (segment (start 79.502 69.977) (end 79.51 69.985) (width 0.25) (layer "F.Cu") (net 26))
+  (segment (start 87.997 68.971) (end 88.011 68.985) (width 0.25) (layer "F.Cu") (net 27))
+  (segment (start 64.145 68.971) (end 87.997 68.971) (width 0.25) (layer "F.Cu") (net 27))
   (zone (net 8) (net_name "GND") (layer "B.Cu") (hatch edge 0.508)
     (connect_pads (clearance 0.508))
-    (min_thickness 0.254)
-    (fill (thermal_gap 0.508) (thermal_bridge_width 0.508))
+    (min_thickness 0.254) (filled_areas_thickness no)
+    (fill yes (thermal_gap 0.508) (thermal_bridge_width 0.508))
     (polygon
       (pts
-        (xy 270.5 131)
-        (xy 21 131)
-        (xy 21 19)
-        (xy 270.5 19)
+        (xy 270.256 131.445)
+        (xy 20.955 131.572)
+        (xy 21.082 19.05)
+        (xy 270.51 19.05)
       )
     )

Commit message: pcb avec bon pin & quartz & régulateur de tension
Parts:
- added C1: 15pF, Capacitor_SMD:C_1206_3216Metric, F.Cu at (90.9, 94.4)
- added C2: 15pF, Capacitor_SMD:C_1206_3216Metric, F.Cu at (90.9, 99.3)
- added C3: C, Capacitor_SMD:C_1206_3216Metric, F.Cu at (102.0, 84.8)
- added C4: C, Capacitor_SMD:C_1206_3216Metric, F.Cu at (94.4, 90.8)
- added U2: LM1117-5.0, eec:National_Semiconductor-LM1117IMP-5.0-Level_A, F.Cu at (94.4, 81.8)
- added Y1: Crystal, Crystal:Resonator-2Pin_W10.0mm_H5.0mm, F.Cu at (98.9, 99.4)
- J1: footprint Connector_PinHeader_1.00mm:PinHeader_1x08_P1.00mm_Vertical -> Connector_PinSocket_2.54mm:PinSocket_1x08_P2.54mm_Vertical
- J2: footprint Connector_PinHeader_1.00mm:PinHeader_1x06_P1.00mm_Vertical -> Connector_PinSocket_2.54mm:PinSocket_1x06_P2.54mm_Vertical
- J3: footprint Connector_PinHeader_1.00mm:PinHeader_1x09_P1.00mm_Vertical -> Connector_PinSocket_2.54mm:PinSocket_1x09_P2.54mm_Vertical
- moved J3 105.1 mm to (141.9, 65.2), turned to 0 degrees
- moved U1 54.0 mm to (110.1, 75.7)
- moved J2 46.8 mm to (134.5, 62.5), turned to -90 degrees
- moved J1 45.3 mm to (136.0, 108.8)
Connections:
- U1 pad 9: unconnected-(U1-Pad9) -> Net-(U1-Pad9)
Routing:
- net VCC: track 0.00 -> 136.8 mm, vias 0 -> 4
- net Net-(J3-Pad6): track 20.2 -> 121.8 mm, vias 0 -> 2
- net Net-(J3-Pad5): track 20.8 -> 85.0 mm, vias 0 -> 2
- net Net-(U1-Pad9): track 0.00 -> 18.5 mm
- net Net-(J1-Pad2): track 29.7 -> 18.3 mm
- net GND: track 0.00 -> 10.6 mm, vias 0 -> 4
- net Net-(J1-Pad5): track 28.7 -> 18.3 mm
- net Net-(J1-Pad3): track 28.5 -> 18.3 mm
- net Net-(J1-Pad4): track 28.0 -> 18.3 mm
- net Net-(C2-Pad1): track 0.00 -> 6.64 mm
- net +6V: track 0.00 -> 3.92 mm
- net Net-(J2-Pad3): track 24.5 -> 27.6 mm, vias 0 -> 2
- net Net-(J2-Pad2): track 23.9 -> 22.4 mm
Other:
- board size 249.5 x 112.5 mm -> 93.1 x 56 mm

Commit message: PCB fini
Parts:
- moved U2 24.1 mm to (117.3, 74.4)
- moved C4 23.5 mm to (117.1, 84.9)
- moved C2 22.8 mm to (113.6, 99.5), turned to 0 degrees
- moved J2 22.8 mm to (157.2, 62.4)
- moved J3 22.8 mm to (164.6, 65.1)
- moved J1 22.8 mm to (158.8, 108.8)
- moved U1 22.8 mm to (132.9, 75.6)
- moved Y1 22.8 mm to (121.7, 99.3)
- moved C1 22.7 mm to (113.5, 94.5), turned to 0 degrees
- moved C3 21.5 mm to (123.2, 81.4)
Connections:
- C1 pad 1: Net-(U1-Pad9) -> GND
- C1 pad 2: unconnected-(C1-Pad2) -> Net-(C1-Pad2)
- C2 pad 1: Net-(C2-Pad1) -> GND
- C2 pad 2: unconnected-(C2-Pad2) -> Net-(C2-Pad2)
- J1 pad 2: Net-(J1-Pad2) -> unconnected-(J1-Pad2)
- J1 pad 3: Net-(J1-Pad3) -> VCC
- J1 pad 5: Net-(J1-Pad5) -> Net-(U1-Pad17)
- J1 pad 6: GND -> Net-(U1-Pad19)
- J1 pad 7: unconnected-(J1-Pad7) -> Net-(U1-Pad18)
- J1 pad 8: VCC -> GND
- U1 pad 10: unconnected-(U1-Pad10) -> Net-(C2-Pad2)
- U1 pad 16: Net-(J1-Pad2) -> unconnected-(U1-Pad16)
- U1 pad 17: Net-(J1-Pad3) -> Net-(U1-Pad17)
- U1 pad 18: Net-(J1-Pad4) -> Net-(U1-Pad18)
- U1 pad 19: Net-(J1-Pad5) -> Net-(U1-Pad19)
- U1 pad 6: unconnected-(U1-Pad6) -> Net-(J1-Pad4)
- U1 pad 9: Net-(U1-Pad9) -> Net-(C1-Pad2)
- Y1 pad 1: Net-(C2-Pad1) -> Net-(C2-Pad2)
- Y1 pad 2: Net-(U1-Pad9) -> Net-(C1-Pad2)
Routing:
- net Net-(J3-Pad6): track 121.8 -> 50.2 mm, vias 2 -> 0
- net Net-(J1-Pad4): track 18.3 -> 88.4 mm
- net VCC: track 136.8 -> 189.3 mm, vias 4 -> 2
- net +6V: track 3.92 -> 52.2 mm
- net GND: track 10.6 -> 54.4 mm, vias 4 -> 5
- net Net-(U1-Pad19): track 0.00 -> 42.6 mm
- net Net-(J3-Pad5): track 85.0 -> 57.8 mm, vias 2 -> 0
- net Net-(U1-Pad18): track 0.00 -> 21.4 mm
- net Net-(U1-Pad17): track 0.00 -> 20.3 mm
- net Net-(C1-Pad2): track 0.00 -> 18.6 mm
- net Net-(U1-Pad9): track 18.5 -> 0.00 mm
- net Net-(J1-Pad5): track 18.3 -> 0.00 mm
- net Net-(J1-Pad3): track 18.3 -> 0.00 mm
- net Net-(J1-Pad2): track 18.3 -> 0.00 mm
- net Net-(C2-Pad2): track 0.00 -> 18.2 mm
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Other:
- board size 93.1 x 56 mm -> 93.1 x 59.5 mm
